Commit message: updated

File: src/my_robot_description/urdf/camer_plugin.urdf.xacro (robot description, xacro)
@@ -7,5 +7,5 @@
       <update_rate>50</update_rate>
       <always_on>true</always_on>
-      <visualize>true</visualize>
+      <visualize>false</visualize>
       <camera_name>my_camera</camera_name>
       <camera>

File: src/my_robot_description/urdf/lidar_plugin.urdf.xacro (robot description, xacro)
@@ -5,6 +5,6 @@
   <sensor name="laser" type='ray'>
     <pose>0 0 0 0 0 0</pose>
-    <update_rate>10</update_rate>
-    <visualize>true</visualize>
+    <update_rate>50</update_rate>
+    <visualize>false</visualize>
     <ray>
       <scan>

File: src/my_robot_description/urdf/my_robot.urdf.xacro (robot description, xacro)
@@ -6,4 +6,5 @@
     </material>
   </xacro:macro>
+  <link name="world_link"/>
   <link name="base_link">
     <visual>
@@ -204,4 +205,8 @@
 </gazebo>
 <!-- - - - - - - - - - - -  - - - - - - - - - - - - - - - - - - - - -  - - - - -->
+<joint name="world_to_base" type="fixed">
+  <parent link="world_link"/>
+  <child link="base_link"/>
+</joint>
 <xacro:macro name="base_connection_joint" params="prefix x y z r p yaw">
    <joint name="base_${prefix}_connection_joint" type="fixed">
@@ -214,9 +219,8 @@
 <xacro:base_connection_joint prefix="r" x="0" y="-0.205" z="0" r="1.57075" p="0" yaw="0"/>
 <xacro:macro name="connection_rocker_joint" params="prefix x y z r p yaw">
-   <joint name="${prefix}_connection_${prefix}_rocker_joint" type="revolute">
+   <joint name="${prefix}_connection_${prefix}_rocker_joint" type="fixed">
   <parent link="${prefix}_connection_link"/>
   <child link="${prefix}_rocker_link"/>
   <axis xyz="0 1 0"/>
-  <limit lower="-0.2" upper="0.2" effort="10" velocity="1.0"/>
   <origin xyz="${x} ${y} ${z}" rpy="${r} ${p} ${yaw}"/>
 </joint>
@@ -332,3 +336,4 @@
 <xacro:include filename='camer_plugin.urdf.xacro'/>
 <xacro:include filename='gazebo_control_plugin.urdf.xacro'/>
+<xacro:include filename = 'depth_camera_plugin.urdf.xacro'/>
 </robot>
